File: Hardware/micromouse.kicad_pcb (KiCad board)
At the start: 2 copper layers, 1 part

Commit message: Added outlines for the board added a basic mace grid into the pcb drawing added sensor positions for the infrared sensors
Parts:
- moved REF** 282.4 mm to (386.0, -46.0)
Other:
- board outline added: 100 x 74 mm
Changed lines of the file:
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@@
-(kicad_pcb (version 20171130) (host pcbnew 5.0.1)
+(kicad_pcb (version 20171130) (host pcbnew "(5.0.1)-4")
   (general
     (thickness 1.6)
-    (drawings 0)
+    (drawings 43)
     (tracks 0)
     (zones 0)
@@
     (nets 1)
   )
-  (page A4)
+  (page A3)
   (layers
     (0 F.Cu signal)
@@
     (36 B.SilkS user)
     (37 F.SilkS user)
-    (38 B.Mask user)
+    (38 B.Mask user hide)
     (39 F.Mask user)
     (40 Dwgs.User user)
@@
     (solder_mask_min_width 0.25)
     (aux_axis_origin 0 0)
-    (visible_elements FFFFFF7F)
+    (grid_origin 300 120)
+    (visible_elements 7FFFFFFF)
     (pcbplotparams
       (layerselection 0x010fc_ffffffff)
@@
   )
   (module Display:Adafruit_SSD1306 (layer F.Cu)
-    (at 130.81 74.93)
+    (at 386 -46)
     (descr "Adafruit SSD1306 OLED 1.3 inch 128x64 I2C & SPI https://learn.adafruit.com/monochrome-oled-breakouts/downloads")
     (tags "Adafruit SSD1306 OLED 1.3 inch 128x64 I2C & SPI ")
@@
     )
   )
+  (dimension 156 (width 0.3) (layer Cmts.User)
+    (gr_text "156,000 mm" (at 300 20.9) (layer Cmts.User)
+      (effects (font (size 1.5 1.5) (thickness 0.3)))
+    )
+    (feature1 (pts (xy 378 30) (xy 378 22.413579)))
+    (feature2 (pts (xy 222 30) (xy 222 22.413579)))
+    (crossbar (pts (xy 222 23) (xy 378 23)))
+    (arrow1a (pts (xy 378 23) (xy 376.873496 23.586421)))
+    (arrow1b (pts (xy 378 23) (xy 376.873496 22.413579)))
+    (arrow2a (pts (xy 222 23) (xy 223.126504 23.586421)))
+    (arrow2b (pts (xy 222 23) (xy 223.126504 22.413579)))
+  )
+  (dimension 180 (width 0.3) (layer Cmts.User)
+    (gr_text "180,000 mm" (at 300 15.9) (layer Cmts.User)
+      (effects (font (size 1.5 1.5) (thickness 0.3)))
+    )
+    (feature1 (pts (xy 390 30) (xy 390 17.413579)))
+    (feature2 (pts (xy 210 30) (xy 210 17.413579)))
+    (crossbar (pts (xy 210 18) (xy 390 18)))
+    (arrow1a (pts (xy 390 18) (xy 388.873496 18.586421)))
+    (arrow1b (pts (xy 390 18) (xy 388.873496 17.413579)))
+    (arrow2a (pts (xy 210 18) (xy 211.126504 18.586421)))
+    (arrow2b (pts (xy 210 18) (xy 211.126504 17.413579)))
+  )
+  (dimension 156 (width 0.3) (layer Cmts.User)
+    (gr_text "156,000 mm" (at 399.1 120 270) (layer Cmts.User)
+      (effects (font (size 1.5 1.5) (thickness 0.3)))
+    )
+    (feature1 (pts (xy 390 198) (xy 397.586421 198)))
+    (feature2 (pts (xy 390 42) (xy 397.586421 42)))
+    (crossbar (pts (xy 397 42) (xy 397 198)))
+    (arrow1a (pts (xy 397 198) (xy 396.413579 196.873496)))
+    (arrow1b (pts (xy 397 198) (xy 397.586421 196.873496)))
+    (arrow2a (pts (xy 397 42) (xy 396.413579 43.126504)))
+    (arrow2b (pts (xy 397 42) (xy 397.586421 43.126504)))
+  )
+  (dimension 180 (width 0.3) (layer Cmts.User)
+    (gr_text "180,000 mm" (at 405.1 120 270) (layer Cmts.User)
+      (effects (font (size 1.5 1.5) (thickness 0.3)))
+    )
+    (feature1 (pts (xy 390 210) (xy 403.586421 210)))
+    (feature2 (pts (xy 390 30) (xy 403.586421 30)))
+    (crossbar (pts (xy 403 30) (xy 403 210)))
+    (arrow1a (pts (xy 403 210) (xy 402.413579 208.873496)))
+    (arrow1b (pts (xy 403 210) (xy 403.586421 208.873496)))
+    (arrow2a (pts (xy 403 30) (xy 402.413579 31.126504)))
+    (arrow2b (pts (xy 403 30) (xy 403.586421 31.126504)))
+  )
+  (gr_line (start 254 95) (end 24 84) (layer Cmts.User) (width 0.2))
+  (gr_line (start 30 45) (end 254 95) (layer Cmts.User) (width 0.2))
+  (gr_line (start 254 145) (end 30 196) (layer Cmts.User) (width 0.2))
+  (gr_line (start 25 156) (end 254 145) (layer Cmts.User) (width 0.2))
+  (gr_arc (start 254 94) (end 30.000001 44.000001) (angle -10.1) (layer Cmts.User) (width 0.2))
+  (gr_arc (start 254 145) (end 25.000001 155.999999) (angle -10) (layer Cmts.User) (width 0.2))
+  (gr_line (start 245 125) (end 198 203) (layer Cmts.User) (width 0.2))
+  (gr_line (start 245 125) (end 184 193) (layer Cmts.User) (width 0.2))
+  (gr_line (start 246 116) (end 198 36) (layer Cmts.User) (width 0.2))
+  (gr_line (start 184 46) (end 246 116) (layer Cmts.User) (width 0.2))
+  (gr_arc (start 245 125) (end 184.000001 192.999999) (angle -10.6) (layer Cmts.User) (width 0.2))
+  (gr_arc (start 245 115) (end 198.000001 36.000001) (angle -10.4) (layer Cmts.User) (width 0.2))
+  (gr_line (start 30 30) (end 390 30) (layer Dwgs.User) (width 0.2))
+  (gr_line (start 273 157) (end 284 157) (layer Edge.Cuts) (width 0.15))
+  (gr_line (start 316 157) (end 327 157) (layer Edge.Cuts) (width 0.15))
+  (gr_arc (start 273 120) (end 273 83) (angle -180) (layer Edge.Cuts) (width 0.15))
+  (gr_line (start 284 83) (end 273 83) (layer Edge.Cuts) (width 0.15))
+  (gr_line (start 284 92) (end 284 83) (layer Edge.Cuts) (width 0.15))
+  (gr_line (start 316 92) (end 284 92) (layer Edge.Cuts) (width 0.15))
+  (gr_line (start 316 83) (end 316 92) (layer Edge.Cuts) (width 0.15))
+  (gr_line (start 327 83) (end 316 83) (layer Edge.Cuts) (width 0.15))
+  (gr_line (start 336 92) (end 327 83) (layer Edge.Cuts) (width 0.15))
+  (gr_line (start 336 148) (end 336 92) (layer Edge.Cuts) (width 0.15))
+  (gr_line (start 327 157) (end 336 148) (layer Edge.Cuts) (width 0.15))
+  (gr_line (start 316 148) (end 316 157) (layer Edge.Cuts) (width 0.15))
+  (gr_line (start 284 148) (end 316 148) (layer Edge.Cuts) (width 0.15))
+  (gr_line (start 284 157) (end 284 148) (layer Edge.Cuts) (width 0.15))
+  (gr_line (start 300 30) (end 300 210) (layer Dwgs.User) (width 0.2))
+  (gr_line (start 30 120) (end 390 120) (layer Dwgs.User) (width 0.2))
+  (gr_line (start 222 210) (end 222 30) (layer Dwgs.User) (width 0.2))
+  (gr_line (start 198 30) (end 198 210) (layer Dwgs.User) (width 0.2))
+  (gr_line (start 42 30) (end 42 210) (layer Dwgs.User) (width 0.2))
+  (gr_line (start 378 30) (end 378 210) (layer Dwgs.User) (width 0.2))
+  (gr_line (start 30 42) (end 390 42) (layer Dwgs.User) (width 0.2))
+  (gr_line (start 30 198) (end 390 198) (layer Dwgs.User) (width 0.2))
+  (gr_line (start 210 30) (end 210 210) (layer Dwgs.User) (width 0.2))
+  (gr_line (start 30 210) (end 30 30) (layer Dwgs.User) (width 0.2))
+  (gr_line (start 390 210) (end 30 210) (layer Dwgs.User) (width 0.2))
+  (gr_line (start 390 30) (end 390 210) (layer Dwgs.User) (width 0.2))
 )
